Commit message: Signed-off-by: Andrea Patrizi <andreapatrizi1b6e6@gmail.com>

File: kyonrlstepping/config/xmj_env_files/kyon_wheels.urdf (robot description, URDF)
Before this commit: robot kyon, 31 links, 30 joints
Joints:
- joint wheel_joint_1: limit effort=132 velocity=15.5 -> effort=132 velocity=60.0
- joint wheel_joint_2: limit effort=132 velocity=15.5 -> effort=132 velocity=60.0
- joint wheel_joint_3: limit effort=132 velocity=15.5 -> effort=132 velocity=60.0
- joint wheel_joint_4: limit effort=132 velocity=15.5 -> effort=132 velocity=60.0
