Commit message: Signed-off-by: Andrea Patrizi <andreapatrizi1b6e6@gmail.com>

File: kyonrlstepping/config/xmj_env_files/kyon.urdf (robot description, URDF)
Before this commit: robot kyon, 26 links, 25 joints
Links:
- added link world
Joints:
- added joint reference: type floating, parent world, child base_link

Commit message: added imu sensors

File: kyonrlstepping/config/xmj_env_files/kyon.urdf (robot description, URDF)
Before this commit: robot kyon, 27 links, 26 joints
Links:
- added link imu_link
Joints:
- added joint imu_joint: type fixed, parent pelvis, child imu_link, origin xyz=0.0 0.0 0.0 rpy=0.0 0.0 0.0
