Commit message: added kyon files for usage with xbot-mujoco

File: kyonrlstepping/config/xmj_env_files/kyon_real/kyon_real_wheels_no_yaw.urdf (robot description, URDF)
Before this commit: robot kyon_real, 24 links, 23 joints
Links:
- added link ankle_yaw_1_link, mass 1.4742389; collision mesh filename=/root/ibrido_ws/src/iit-kyon-description/kyon_urdf/meshes/c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 scale=0.001 0.001 0.001; visual mesh filename=/root/ibrido_ws/src/iit-kyon-description/kyon_urdf/meshes/m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 scale=0.001 0.001 0.001
- added link ankle_yaw_2_link, mass 1.4742389; collision mesh filename=/root/ibrido_ws/src/iit-kyon-description/kyon_urdf/meshes/c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 scale=0.001 0.001 0.001; visual mesh filename=/root/ibrido_ws/src/iit-kyon-description/kyon_urdf/meshes/m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 scale=0.001 0.001 0.001
- added link ankle_yaw_3_link, mass 1.4742389; collision mesh filename=/root/ibrido_ws/src/iit-kyon-description/kyon_urdf/meshes/c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 scale=0.001 0.001 0.001; visual mesh filename=/root/ibrido_ws/src/iit-kyon-description/kyon_urdf/meshes/m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 scale=0.001 0.001 0.001
- added link ankle_yaw_4_link, mass 1.4742389; collision mesh filename=/root/ibrido_ws/src/iit-kyon-description/kyon_urdf/meshes/c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 scale=0.001 0.001 0.001; visual mesh filename=/root/ibrido_ws/src/iit-kyon-description/kyon_urdf/meshes/m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 scale=0.001 0.001 0.001
- added link ball_1
- added link ball_2
- added link ball_3
- added link ball_4
- added link wheel_1, mass 1.1618108; collision cylinder length=0.05 radius=0.1066; visual mesh filename=/root/ibrido_ws/src/iit-kyon-description/kyon_urdf/meshes/m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 scale=0.001 0.001 0.001
- added link wheel_2, mass 1.1618108; collision cylinder length=0.05 radius=0.1066; visual mesh filename=/root/ibrido_ws/src/iit-kyon-description/kyon_urdf/meshes/m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 scale=0.001 0.001 0.001
- added link wheel_3, mass 1.1618108; collision cylinder length=0.05 radius=0.1066; visual mesh filename=/root/ibrido_ws/src/iit-kyon-description/kyon_urdf/meshes/m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 scale=0.001 0.001 0.001
- added link wheel_4, mass 1.1618108; collision cylinder length=0.05 radius=0.1066; visual mesh filename=/root/ibrido_ws/src/iit-kyon-description/kyon_urdf/meshes/m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 scale=0.001 0.001 0.001
- link knee_pitch_1_link: mass 0.70900216 -> 1.5279917; geometry collision mesh filename=/root/ibrido_ws/src/iit-kyon-description/kyon_urdf/meshes/c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 scale=0.001 0.001 0.001; visual mesh filename=/root/ibrido_ws/src/iit-kyon-description/kyon_urdf/meshes/m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 scale=0.001 0.001 0.001
- link knee_pitch_2_link: mass 0.70900216 -> 1.5279917
- link knee_pitch_3_link: mass 0.70900216 -> 1.5279917; geometry collision mesh filename=/root/ibrido_ws/src/iit-kyon-description/kyon_urdf/meshes/c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 scale=0.001 0.001 0.001; visual mesh filename=/root/ibrido_ws/src/iit-kyon-description/kyon_urdf/meshes/m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 scale=0.001 0.001 0.001
- link knee_pitch_4_link: mass 0.70900216 -> 1.5279917
Joints:
- removed joint contact_1_joint
- removed joint contact_2_joint
- removed joint contact_3_joint
- removed joint contact_4_joint
- added joint ankle_yaw_1: type revolute, parent knee_pitch_1_link, child ankle_yaw_1_link, origin xyz=0.0 -0.0735 0.059000000000000004 rpy=-1.57079632679 0.0 0.0, axis 0 0 1, limit lower=-3.0 upper=3.0 effort=185 velocity=7.6
- added joint ankle_yaw_2: type revolute, parent knee_pitch_2_link, child ankle_yaw_2_link, origin xyz=0.0 -0.0735 0.059000000000000004 rpy=-1.57079632679 0.0 0.0, axis 0 0 1, limit lower=-3.0 upper=3.0 effort=185 velocity=7.6
- added joint ankle_yaw_3: type revolute, parent knee_pitch_3_link, child ankle_yaw_3_link, origin xyz=0.0 -0.0735 0.059000000000000004 rpy=-1.57079632679 0.0 0.0, axis 0 0 1, limit lower=-3.0 upper=3.0 effort=185 velocity=7.6
- added joint ankle_yaw_4: type revolute, parent knee_pitch_4_link, child ankle_yaw_4_link, origin xyz=0.0 -0.0735 0.059000000000000004 rpy=-1.57079632679 0.0 0.0, axis 0 0 1, limit lower=-3.0 upper=3.0 effort=185 velocity=7.6
- added joint ball_joint_1: type fixed, parent ankle_yaw_1_link, child ball_1, origin xyz=0.0 0.0 -0.2205 rpy=-1.57079632679 0.0 0.0
- added joint ball_joint_2: type fixed, parent ankle_yaw_2_link, child ball_2, origin xyz=0.0 0.0 -0.2205 rpy=-1.57079632679 0.0 0.0
- added joint ball_joint_3: type fixed, parent ankle_yaw_3_link, child ball_3, origin xyz=0.0 0.0 -0.2205 rpy=-1.57079632679 0.0 0.0
- added joint ball_joint_4: type fixed, parent ankle_yaw_4_link, child ball_4, origin xyz=0.0 0.0 -0.2205 rpy=-1.57079632679 0.0 0.0
- added joint contact_joint_1: type fixed, parent ankle_yaw_1_link, child contact_1, origin xyz=0.0753775 0.0  -0.2958775  rpy=0.0 -0.785 0.0
- added joint contact_joint_2: type fixed, parent ankle_yaw_2_link, child contact_2, origin xyz=-0.0753775 0.0  -0.2958775  rpy=0.0 0.785 0.0
- added joint contact_joint_3: type fixed, parent ankle_yaw_3_link, child contact_3, origin xyz=0.0753775 0.0  -0.2958775  rpy=0.0 -0.785 0.0
- added joint contact_joint_4: type fixed, parent ankle_yaw_4_link, child contact_4, origin xyz=-0.0753775 0.0  -0.2958775  rpy=0.0 0.785 0.0
- added joint wheel_joint_1: type continuous, parent ankle_yaw_1_link, child wheel_1, origin xyz=0.0 0.0 -0.2205 rpy=-1.57079632679 0.0 0.0, axis 0 0 1, limit lower=-1e9 upper=1e9 effort=100 velocity=30
- added joint wheel_joint_2: type continuous, parent ankle_yaw_2_link, child wheel_2, origin xyz=0.0 0.0 -0.2205 rpy=-1.57079632679 0.0 0.0, axis 0 0 1, limit lower=-1e9 upper=1e9 effort=100 velocity=30
- added joint wheel_joint_3: type continuous, parent ankle_yaw_3_link, child wheel_3, origin xyz=0.0 0.0 -0.2205 rpy=-1.57079632679 0.0 0.0, axis 0 0 1, limit lower=-1e9 upper=1e9 effort=100 velocity=30
- added joint wheel_joint_4: type continuous, parent ankle_yaw_4_link, child wheel_4, origin xyz=0.0 0.0 -0.2205 rpy=-1.57079632679 0.0 0.0, axis 0 0 1, limit lower=-1e9 upper=1e9 effort=100 velocity=30
