Commit message: Signed-off-by: Andrea Patrizi <andreapatrizi1b6e6@gmail.com>

File: kyonrlstepping/config/xmj_env_files/kyon_real/kyon_real_wheels.urdf (robot description, URDF)
Before this commit: robot kyon_real, 36 links, 35 joints
Links:
- added link world
Joints:
- added joint reference: type floating, parent world, child pelvis
