Commit message: Update Kyon XMJ launch and impedance configs

File: kyonrlstepping/config/xmj_env_files/kyon_real/kyon_real_no_wheels.urdf (robot description, URDF)
Before this commit: robot kyon_real, 25 links, 24 joints
Links:
- added link battery, mass 9.8; visual box size=0.329 0.225 0.0793
- link hip_roll_1_link: geometry visual mesh filename=/root/ibrido_ws/src/iit-kyon-description/kyon_urdf/meshes/m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 scale=0.001 -0.001 0.001
- link hip_roll_2_link: geometry visual mesh filename=/root/ibrido_ws/src/iit-kyon-description/kyon_urdf/meshes/m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 scale=0.001 0.001 0.001
- link hip_roll_3_link: geometry visual mesh filename=/root/ibrido_ws/src/iit-kyon-description/kyon_urdf/meshes/m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 scale=0.001 -0.001 0.001
- link hip_roll_4_link: geometry visual mesh filename=/root/ibrido_ws/src/iit-kyon-description/kyon_urdf/meshes/m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 scale=0.001 0.001 0.001
- link knee_pitch_1_link: geometry collision mesh filename=/root/ibrido_ws/src/iit-kyon-description/kyon_urdf/meshes/c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 scale=0.001 0.001 0.001; visual mesh filename=/root/ibrido_ws/src/iit-kyon-description/kyon_urdf/meshes/m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 scale=0.001 0.001 0.001
- link knee_pitch_3_link: geometry collision mesh filename=/root/ibrido_ws/src/iit-kyon-description/kyon_urdf/meshes/c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 scale=0.001 0.001 0.001; visual mesh filename=/root/ibrido_ws/src/iit-kyon-description/kyon_urdf/meshes/m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 scale=0.001 0.001 0.001
Joints:
- added joint battery_joint: type fixed, parent pelvis, child battery, origin xyz=0.0 0.0 -0.02725

File: kyonrlstepping/config/xmj_env_files/kyon_real/kyon_real_wheels.urdf (robot description, URDF)
Before this commit: robot kyon_real, 37 links, 36 joints
Links:
- added link battery, mass 9.8; visual box size=0.329 0.225 0.0793
- link hip_roll_1_link: geometry visual mesh filename=/root/ibrido_ws/src/iit-kyon-description/kyon_urdf/meshes/m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 scale=0.001 -0.001 0.001
- link hip_roll_2_link: geometry visual mesh filename=/root/ibrido_ws/src/iit-kyon-description/kyon_urdf/meshes/m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 scale=0.001 0.001 0.001
- link hip_roll_3_link: geometry visual mesh filename=/root/ibrido_ws/src/iit-kyon-description/kyon_urdf/meshes/m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 scale=0.001 -0.001 0.001
- link hip_roll_4_link: geometry visual mesh filename=/root/ibrido_ws/src/iit-kyon-description/kyon_urdf/meshes/m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 scale=0.001 0.001 0.001
- link wheel_1: geometry collision cylinder length=0.03 radius=0.1066; visual mesh filename=/root/ibrido_ws/src/iit-kyon-description/kyon_urdf/meshes/m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 scale=0.001 0.001 0.001
- link wheel_2: geometry collision cylinder length=0.03 radius=0.1066; visual mesh filename=/root/ibrido_ws/src/iit-kyon-description/kyon_urdf/meshes/m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 scale=0.001 0.001 0.001
- link wheel_3: geometry collision cylinder length=0.03 radius=0.1066; visual mesh filename=/root/ibrido_ws/src/iit-kyon-description/kyon_urdf/meshes/m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 scale=0.001 0.001 0.001
- link wheel_4: geometry collision cylinder length=0.03 radius=0.1066; visual mesh filename=/root/ibrido_ws/src/iit-kyon-description/kyon_urdf/meshes/m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 scale=0.001 0.001 0.001
Joints:
- added joint battery_joint: type fixed, parent pelvis, child battery, origin xyz=0.0 0.0 -0.02725
