Commit message: Signed-off-by: Andrea Patrizi <andreapatrizi1b6e6@gmail.com>

File: kyonrlstepping/config/xmj_env_files/b2w/unitree_b2w.urdf (robot description, URDF)
Before this commit: robot unitree_b2w, 39 links, 38 joints
Links:
- removed link world
Joints:
- removed joint reference

Commit message: fixed urdf + added missing homing cfgs

File: kyonrlstepping/config/xmj_env_files/b2w/unitree_b2w.urdf (robot description, URDF)
Before this commit: robot unitree_b2w, 38 links, 37 joints
Links:
- link FL_calf: geometry collision box size=0.05 0.028 0.035; collision box size=0.1 0.0245 0.018
- link FL_foot: geometry collision cylinder length=0.03 radius=0.1125; visual mesh filename=/root/ibrido_ws/src/unitree_ros/robots/b2w_description/mesh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
- link FL_hip: geometry collision cylinder length=0.05 radius=0.07; visual mesh filename=/root/ibrido_ws/src/unitree_ros/robots/b2w_description/mesh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 scale=1 1 1
- link FL_thigh: geometry collision box size=0.32 0.0455 0.054; visual mesh filename=/root/ibrido_ws/src/unitree_ros/robots/b2w_description/mesh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 scale=1 1 1
- link FR_calf: geometry collision box size=0.05 0.028 0.035; collision box size=0.1 0.0245 0.018
- link FR_foot: geometry collision cylinder length=0.03 radius=0.1125; visual mesh filename=/root/ibrido_ws/src/unitree_ros/robots/b2w_description/mesh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
- link FR_hip: geometry collision cylinder length=0.05 radius=0.07; visual mesh filename=/root/ibrido_ws/src/unitree_ros/robots/b2w_description/mesh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 scale=1 1 1
- link FR_thigh: geometry collision box size=0.32 0.0455 0.054; visual mesh filename=/root/ibrido_ws/src/unitree_ros/robots/b2w_description/mesh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 scale=1 1 1
- link RL_calf: geometry collision box size=0.05 0.028 0.035; collision box size=0.1 0.0245 0.018
- link RL_foot: geometry collision cylinder length=0.03 radius=0.1125; visual mesh filename=/root/ibrido_ws/src/unitree_ros/robots/b2w_description/mesh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
- link RL_hip: geometry collision cylinder length=0.05 radius=0.07; visual mesh filename=/root/ibrido_ws/src/unitree_ros/robots/b2w_description/mesh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 scale=1 1 1
- link RL_thigh: geometry collision box size=0.32 0.0455 0.054; visual mesh filename=/root/ibrido_ws/src/unitree_ros/robots/b2w_description/mesh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 scale=1 1 1
- link RR_calf: geometry collision box size=0.05 0.028 0.035; collision box size=0.1 0.0245 0.018
- link RR_foot: geometry collision cylinder length=0.03 radius=0.1125; visual mesh filename=/root/ibrido_ws/src/unitree_ros/robots/b2w_description/mesh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
- link RR_hip: geometry collision cylinder length=0.05 radius=0.07; visual mesh filename=/root/ibrido_ws/src/unitree_ros/robots/b2w_description/mesh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 scale=1 1 1
- link RR_thigh: geometry collision box size=0.32 0.0455 0.054; visual mesh filename=/root/ibrido_ws/src/unitree_ros/robots/b2w_description/mesh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 scale=1 1 1
- link lidar_link: mass 6.55E-08 -> 1E-03
- link trunk: geometry collision box size=0.5 0.28 0.15; visual mesh filename=/root/ibrido_ws/src/unitree_ros/robots/b2w_description/mesh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 scale=1 1 1

Commit message: big bfix in kyon and b2w configs: typo after horizon refactor, causing v and a reg to be just on 1st node -> MPCs diverged

File: kyonrlstepping/config/xmj_env_files/b2w/unitree_b2w.urdf (robot description, URDF)
Before this commit: robot unitree_b2w, 38 links, 37 joints
Links:
- link FL_foot: geometry collision cylinder length=0.05 radius=0.1129; visual mesh filename=/root/ibrido_ws/src/unitree_ros/robots/b2w_description/mesh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
- link FR_foot: geometry collision cylinder length=0.05 radius=0.1129; visual mesh filename=/root/ibrido_ws/src/unitree_ros/robots/b2w_description/mesh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
- link RL_foot: geometry collision cylinder length=0.05 radius=0.1129; visual mesh filename=/root/ibrido_ws/src/unitree_ros/robots/b2w_description/mesh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
- link RR_foot: geometry collision cylinder length=0.05 radius=0.1129; visual mesh filename=/root/ibrido_ws/src/unitree_ros/robots/b2w_description/mesh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
